File: KiCad/Star CAN Board.sch (KiCad schematic (older format))
At the start: 4 parts, among them J1 Conn_01x20_Female, J2 Conn_01x02_Male, J3 Conn_01x20_Female

Commit message: hi this is FizzyApple12 pushing stuff for GraveFurball ok bye
Parts:
- R1: footprint Resistor_SMD:R_0603_1608Metric_Pad1.05x0.95mm_HandSolder -> Resistor_THT:R_Axial_DIN0207_L6.3mm_D2.5mm_P10.16mm_Horizontal
Changed lines of the file:
@@
 F 0 "R1" V 5093 2250 50  0000 C CNN
 F 1 "120" V 5184 2250 50  0000 C CNN
-F 2 "Resistor_SMD:R_0603_1608Metric_Pad1.05x0.95mm_HandSolder" V 5230 2250 50  0001 C CNN
+F 2 "Resistor_THT:R_Axial_DIN0207_L6.3mm_D2.5mm_P10.16mm_Horizontal" V 5230 2250 50  0001 C CNN
 F 3 "~" H 5300 2250 50  0001 C CNN
 	1    5300 2250
